Commit message: URDF tweaks. Still requires a lot of cleanup

File: grizzly_description/urdf/base.urdf.xacro (robot description, xacro)
@@ -86,5 +86,5 @@
     </gazebo>
     <joint name="base_footprint_joint" type="fixed">
-		<origin xyz="0 0 ${wheel_x_size/2 - base_z_origin_to_wheel_origin - base_z_origin_offset - base_z_origin_offset}" rpy="0 0 0" />
+		<origin xyz="0 0 ${wheel_x_size/2}" rpy="0 0 0" />
         <parent link="base_footprint"/>
         <child link="base_link" />

File: grizzly_description/urdf/base_yor08.urdf.xacro (robot description, xacro)
@@ -44,17 +44,17 @@
     <!-- Bumblebee -->
     <grizzly_tf parent="base_link" name="bumblebee"
-          translateX="0.24" translateY="0.0" translateZ="${0.4 + base_z_origin_offset}"
+          translateX="0.24" translateY="0.0" translateZ="${0.31 + 0.3 + base_z_origin_offset}"
           rotateX="0.0" rotateY="0.0" rotateZ="0.0"/>
     <!-- Velodyne -->
     <grizzly_tf parent="base_link" name="velodyne"
-          translateX="0.24" translateY="0.0" translateZ="${0.54 + base_z_origin_offset}"
+          translateX="0.24" translateY="0.0" translateZ="${0.55 + 0.3 + base_z_origin_offset}"
           rotateX="0.0" rotateY="0.0" rotateZ="0.0"/>
     <!-- Smart V1-G -->
     <grizzly_tf parent="base_link" name="gps"
           translateX="0.24" translateY="0.24" translateZ="${0.54 + base_z_origin_offset}"
-          rotateX="0.0" rotateY="0.0" rotateZ="0.0"/>
+          rotateX="0.0" rotateY="-0.0" rotateZ="0.0"/>
     <!-- LMS151 -->
-    <grizzly_tf parent="base_link" name="sick"
-          translateX="0.8" translateY="0.0" translateZ="${0.35 + base_z_origin_offset}"
-          rotateX="0.0" rotateY="0.0" rotateZ="0.0"/>
+    <grizzly_tf parent="base_link" name="laser"
+          translateX="0.8" translateY="0.0" translateZ="${0.05 + 0.3 + base_z_origin_offset}"
+          rotateX="0.0" rotateY="0.25" rotateZ="0.0"/>
 </robot>

File: grizzly_description/urdf/sensor_tfs.urdf.xacro (robot description, xacro)
@@ -47,7 +47,7 @@
 		            rpy="${rotateX} ${rotateY} ${rotateZ}" />
 		    <parent link="${parent}" />
-		    <child link="${parent}_${name}_tf" />
+		    <child link="${name}" />
 		</joint>
-		<link name="${parent}_${name}_tf">
+		<link name="${name}">
 			<inertial>
 				<mass value="${mass}" />
